File: hardware/famicom_adapter/famicom_adapter.kicad_sch (KiCad schematic)
At the start: 3 parts, among them J1 CART SLOT TOP ROW, J2 CART SLOT BOTTOM ROW, U1 FC_Slot

Commit message: Fix PCB errors
Other:
- title: OSCR MEGADRIVE ADAPTER -> OSCR FAMICOM ADAPTER
Changed lines of the file:
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@@
   (paper "A4")
   (title_block
-    (title "OSCR MEGADRIVE ADAPTER")
-    (date "2021-11-15")
+    (title "OSCR FAMICOM ADAPTER")
+    (date "2021-11-22")
     (rev "V1")
   )
