File: hardware/mastersystem_adapter/mastersystem_adapter.kicad_sch (KiCad schematic)
At the start: 3 parts, among them J1 CART SLOT TOP ROW, J2 CART SLOT BOTTOM ROW, U1 SMS_Slot

Commit message: Fix PCB errors
Other:
- title: OSCR MEGADRIVE ADAPTER -> OSCR MASTER SYSTEM ADAPTER
Changed lines of the file:
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@@
   (paper "A4")
   (title_block
-    (title "OSCR MEGADRIVE ADAPTER")
-    (date "2021-11-15")
+    (title "OSCR MASTER SYSTEM ADAPTER")
+    (date "2021-11-22")
     (rev "V1")
   )
