File: hardware/snes_adapter/snes_adapter.kicad_pcb (KiCad board)
At the start: 2 copper layers, 96.6 x 25.5 mm, 8 parts, among them J1 CART SLOT TOP ROW, J2 CART SLOT BOTTOM ROW, J3 SNES_Slot, SW1 SW_SPDT, U1 PIC12F629-IP

Commit message: Update SNES adapter
Parts:
- removed C1: C_Small, Capacitor_SMD:C_0805_2012Metric_Pad1.18x1.45mm_HandSolder
- removed JP1, JP2: SolderJumper_2_Open, Jumper:SolderJumper-2_P1.3mm_Open_Pad1.0x1.5mm
- removed SW1: SW_SPDT, Button_Switch_THT:SW_CuK_OS102011MA1QN1_SPDT_Angled
- removed U1: PIC12F629-IP, Package_SO:SOIC-8_3.9x4.9mm_P1.27mm
- added JCIC1: Conn_01x08, Connector_PinHeader_2.54mm:PinHeader_1x08_P2.54mm_Vertical, B.Cu at (178.4, 85.8)
Connections:
- J1 pad 2: +3V3 -> unconnected-(J1-Pad2)
- J1 pad 3: +5V -> VCC
Routing:
- net +5V: track 31.8 -> 0.00 mm, vias 1 -> 0
- net CIC DATA 1: track 33.6 -> 11.5 mm, vias 0 -> 1
- net CIC DATA 0: track 29.6 -> 8.54 mm, vias 1 -> 0
- net CIC RESET: track 30.9 -> 11.1 mm, vias 2 -> 0
- net D40: track 77.8 -> 59.7 mm
- net D41: track 80.7 -> 62.6 mm, vias 3 -> 0
- net CLK2: track 37.0 -> 23.1 mm, vias 2 -> 0
- net VCC: track 130.5 -> 116.9 mm
- net +3V3: track 11.9 -> 0.00 mm
- net GND: track 114.4 -> 104.2 mm
- net A5: track 40.8 -> 31.0 mm, vias 0 -> 1
- net D30: track 10.7 -> 19.6 mm
- net A9: track 25.0 -> 16.3 mm, vias 0 -> 1
- net D14: track 32.2 -> 24.4 mm, vias 0 -> 1
- net A11: track 31.9 -> 24.1 mm
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Other:
- board text added: "CLK"
- board text added: "CR"
- board text added: "WR"
- board text removed: "/WRITE"
- board text removed: "100nF"
- board text removed: "3V"
- board text removed: "3V3"
- board text removed: "CIC"
- board text removed: "CIC CLK"
- board text removed: "CPU CLK"
