File: hardware/snes_adapter/snes_adapter.kicad_sch (KiCad schematic)
At the start: 8 parts, among them J1 CART SLOT TOP ROW, J2 CART SLOT BOTTOM ROW, J3 SNES_Slot, SW1 SW_SPDT, U1 PIC12F629-IP

Commit message: Update SNES adapter
Parts:
- removed C1: C_Small, symbol Device:C_Small
- removed JP1, JP2: SolderJumper_2_Open, symbol Jumper:SolderJumper_2_Open
- removed SW1: SW_SPDT, symbol Switch:SW_SPDT
- removed U1: PIC12F629-IP, Package_DIP:DIP-8_W7.62mm, symbol MCU_Microchip_PIC12:PIC12F629-IP
- added JCIC1: Conn_01x08, symbol Connector_Generic:Conn_01x08
Connections:
- net VCC is gone; now on net +5V: J1.1 (Pin_1), J2.36 (Pin_36), J3.27 (VCC), J3.58 (VCC)
- net +5V: now also JCIC1.1 (Pin_1)
- net CIC DATA 0: now also JCIC1.7 (Pin_7)
- net CIC DATA 1: now also JCIC1.6 (Pin_6)
- net CIC RESET: now also JCIC1.5 (Pin_5)
- net CLK2: now also JCIC1.2 (Pin_2)
- net D40: now also JCIC1.4 (Pin_4)
- net D41: now also JCIC1.3 (Pin_3)
- net GND: now also JCIC1.8 (Pin_8)
- net +3V3: no longer names the net of J1.2 (Pin_2)
- no-connect marks 15 -> 16
